File: SeniorDesign.kicad_sch (KiCad schematic)
At the start: 41 parts, among them J1 USB_B_Micro, J2 Conn_01x04_Pin, J3 Conn_01x04_Pin, J4 Barrel_Jack, SW1 SW_SPDT, U1 STM32F103C8Tx, U2 AMS1117-3.3, U3 LM7812_TO220, U4 XL1509-5.0, Y1 16MHz

Commit message: commit
Parts:
- added C23, C25: 10u, symbol Device:C
- added C24, C26: 10u, symbol Device:C_Polarized
- added D3: 1N4007, Diode_THT:D_DO-41_SOD81_P10.16mm_Horizontal, symbol Diode:1N4007
- added RV1: 10k, symbol Device:R_Potentiometer
- added U5: BUF634P, BUF634P:DIP794W45P254L959H508Q8, symbol BUF634P:BUF634P
- added U6, U7: TL7660IP, TL7660IP:DIP794W45P254L959H508Q8, symbol TL7660IP:TL7660IP
Connections:
- net +12V: now also D3.2 (A), RV1.3, U5.7 (V+)
- net GND: now also C24.1, C26.1, RV1.2, U5.4 (V-), U6.3 (GND), U7.8 (VCC)
- net at C14.1, C15.1, C16.1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: now also D3.1 (K)
- new net: C25.1, U7.2 (CAP+)
- new net: C24.2, C25.2, U6.5 (VOUT), U7.3 (GND), U7.4 (CAP-)
- new net: C23.1, U6.2 (CAP+)
- new net: C23.2, U6.4 (CAP-)
- new net: RV1.1, U5.3 (VIN)
- new net +6V: U5.6 (VO), U6.8 (VCC)
- new net -12V: C26.2, U7.5 (VOUT)
- no-connect marks 28 -> 33
Other:
- note added: "Active Voltage Divider"
- note added: "Power Supply"
- note added: "Voltage Converter"
- note removed: "Analog Power Supply"
- note removed: "Digital Power Supply"
- moved on the sheet: C1, C10, C11, C12, C13, C14, C15, C16, C17, C18, C19, C2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

Commit message: Add co-author
Other:
- company: Michael Mederos -> Michael Mederos and Julio Barreto Tannoux
Changed lines of the file:
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@@
     (title "Senior Design")
     (date "2023-09-18")
-    (company "Michael Mederos")
+    (company "Michael Mederos and Julio Barreto Tannoux")
   )
   (junction (at 161.29 38.1) (diameter 0) (color 0 0 0 0)

Commit message: 10/17/2023
Parts:
- removed C23, C25: 10u, symbol Device:C
- removed C26: 10u, symbol Device:C_Polarized
- removed J4: Barrel_Jack, symbol Connector:Barrel_Jack
- removed RV1: 10k, symbol Device:R_Potentiometer
- removed U5: BUF634P, BUF634P:DIP794W45P254L959H508Q8, symbol BUF634P:BUF634P
- removed U6, U7: TL7660IP, TL7660IP:DIP794W45P254L959H508Q8, symbol TL7660IP:TL7660IP
- added C23: 10u, symbol Device:C_Polarized
- added D4: 1N5226, symbol Device:D_Zener
- added J4: 691243300007, 691243300007:691243300007, symbol 691243300007:691243300007
- added J5: XLR6, symbol Connector_Audio:XLR6
- added R6: 27k, symbol Device:R
- added R7: 10k, symbol Device:R
- added U5: L7912, symbol Regulator_Linear:L7912
- added U6: CD4051B, symbol Analog_Switch:CD4051B
Connections:
- net +3.3VA is gone; now on net +3V3: C6.1, C7.1, FB1.1, U1.9 (VDDA)
- net +12V: now also R6.1, U6.16 (VDD)
- net +3V3: now also D4.1 (K), R6.2, R7.1
- net -12V: now also C24.2, U5.3 (VO)
- net GND: now also C23.1, D4.2 (A), J4.7, J5.2 (P2), R7.2, U5.1 (GND), U6.2 (X6), U6.4 (X7), U6.6 (INH), U6.7 (VEE), U6.8 (VSS)
- net +15V: now reaches C14.1, C15.1, C16.1, D3.1 (K), U3.1 (VI)
- net +15V: now also J5.6 (P6)
- new net -15V: C23.2, J5.4 (P3), U5.2 (VI)
- new net CurrSensor_1: J4.1, U6.13 (X0)
- new net CurrSensor_2: J4.2, U6.14 (X1)
- new net CurrSensor_3: J4.3, U6.15 (X2)
- new net CurrSensor_4: J4.4, U6.12 (X3)
- new net CurrSensor_5: J4.5, U6.1 (X4)
- new net CurrSensor_6: J4.6, U6.5 (X5)
- no-connect marks 33 -> 31
Other:
- note added: "+12V Regulated Voltage"
- note added: "+3.3V Regulated Voltage"
- note added: "-12V Regulated Voltage"
- note added: "NOTE: Check application notes for resistor"
- note removed: "Active Voltage Divider"
- note removed: "Voltage Converter"
- moved on the sheet: C12, C13, C14, C15, C16, C17, C18, C19, C20, C21, C22, D1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

Commit message: 10/18/2023
Parts:
- added C25: C, symbol Device:C
Changed lines of the file:
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@@
+    )
+  )
+  (symbol (lib_id "Device:C") (at 109.22 157.48 0) (unit 1)
+    (in_bom yes) (on_board yes) (dnp no) (fields_autoplaced)
+    (property "Reference" "C25" (at 113.03 156.21 0)
+      (effects (font (size 1.27 1.27)) (justify left))
+    )
+    (property "Value" "C" (at 113.03 158.75 0)
+      (effects (font (size 1.27 1.27)) (justify left))
+    )
+    (property "Footprint" "" (at 110.1852 161.29 0)
+      (effects (font (size 1.27 1.27)) hide)
+    )
+    (property "Datasheet" "~" (at 109.22 157.48 0)
+      (effects (font (size 1.27 1.27)) hide)
+    )
+    (pin "1")
+    (pin "2")
+    (instances
+      (project "SeniorDesign"
+        (path "/24e33b4c-59d4-4763-9563-27915517cfab"
+          (reference "C25") (unit 1)
+        )
+      )
     )
   )
