File: SeniorDesign.kicad_sch (KiCad schematic)
At the start: 50 parts, among them J1 USB_B_Micro, J2 Conn_01x04_Pin, J3 Conn_01x04_Pin, J4 691243300007, J5 XLR6, SW1 SW_SPDT, U1 STM32F103C8Tx, U2 AMS1117-3.3, U3 LM7812_TO220, U4 XL1509-5.0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

Commit message: Julio commit 10/18
Parts:
- added R8: R, symbol Device:R
Changed lines of the file:
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@@
+    )
+  )
+  (symbol (lib_id "Device:R") (at 102.87 153.67 0) (unit 1)
+    (in_bom yes) (on_board yes) (dnp no) (fields_autoplaced)
+    (property "Reference" "R8" (at 105.41 152.4 0)
+      (effects (font (size 1.27 1.27)) (justify left))
+    )
+    (property "Value" "R" (at 105.41 154.94 0)
+      (effects (font (size 1.27 1.27)) (justify left))
+    )
+    (property "Footprint" "" (at 101.092 153.67 90)
+      (effects (font (size 1.27 1.27)) hide)
+    )
+    (property "Datasheet" "~" (at 102.87 153.67 0)
+      (effects (font (size 1.27 1.27)) hide)
+    )
+    (pin "1")
+    (pin "2")
+    (instances
+      (project "SeniorDesign"
+        (path "/24e33b4c-59d4-4763-9563-27915517cfab"
+          (reference "R8") (unit 1)
+        )
+      )
     )
   )
