File: SeniorDesign.kicad_sch (KiCad schematic)
At the start: 52 parts, among them J1 USB_B_Micro, J2 Conn_01x04_Pin, J3 Conn_01x04_Pin, J4 691243300007, J5 XLR6, SW1 SW_SPDT, U1 STM32F103C8Tx, U2 AMS1117-3.3, U3 LM7812_TO220, U4 XL1509-5.0, U5 L7912, U6 CD4051B, Y1 16MHz

Commit message: 10/18/2023
Parts:
- removed C12, C13: 22u, symbol Device:C
- removed C18, C19: 220u, symbol Device:C_Polarized
- removed C20, C22: 10u, symbol Device:C
- removed C21: 180u, symbol Device:C_Polarized
- removed C25: C, symbol Device:C
- removed D1: RED, symbol Device:LED
- removed D2: 1N5820, Diode_THT:D_DO-201AD_P15.24mm_Horizontal, symbol Diode:1N5820
- removed D4: 1N5226, symbol Device:D_Zener
- removed L1: 68u, symbol Device:L
- removed R3: 1k5, symbol Device:R
- removed R8: R, symbol Device:R
- removed U2: AMS1117-3.3, Package_TO_SOT_SMD:SOT-223-3_TabPin2, symbol Regulator_Linear:AMS1117-3.3
- removed U4: XL1509-5.0, Package_SO:SOIC-8_3.9x4.9mm_P1.27mm, symbol Regulator_Switching:XL1509-5.0
- added D1: 1N4007, Diode_THT:D_DO-41_SOD81_P10.16mm_Horizontal, symbol Diode:1N4007
- added D2: 1N4728A, Diode_THT:D_DO-41_SOD81_P10.16mm_Horizontal, symbol Diode:1N47xxA
Connections:
- net +3V3: now also D2.1 (K)
- net -15V: now also D1.1 (K); no longer U5.2 (VI)
- net GND: now also D2.2 (A)
- new net: D1.2 (A), U5.2 (VI)

Commit message: Test
Parts:
- added C12: C, symbol Device:C
- added J6: 691243300007, 691243300007:691243300007, symbol 691243300007:691243300007
- added U2: CD4051B, symbol Analog_Switch:CD4051B
- D2: value 1N4728A -> 1N47xxA
Connections:
- net ADC1_IN3 is gone; now on net UART_RX: U1.13 (PA3)
- net +12V: now also U2.16 (VDD)
- net -12V: now also U2.7 (VEE)
- net GND: now also U2.2 (X6), U2.4 (X7), U2.6 (INH), U2.8 (VSS)
- net UART_RX: now also J3.2 (Pin_2); no longer J3.3 (Pin_3), U1.43 (PB7)
- net UART_TX: now also J3.3 (Pin_3), U1.12 (PA2); no longer J3.2 (Pin_2), U1.42 (PB6)
- net TIM2_CH1: now reaches U1.10 (PA0)
- net ADC2_IN9: now reaches U1.19 (PB1)
- net GPIO_A: now reaches U1.39 (PB3)
- net GPIO_A: now also U2.11 (A)
- net GPIO_B: now reaches U1.40 (PB4)
- net GPIO_B: now also U2.10 (B)
- net GPIO_C: now reaches U1.41 (PB5)
- net GPIO_C: now also U2.9 (C)
- net ADC2_IN6 renamed ADC1_IN6
- new net VoltSensor_1: J6.1, U2.13 (X0)
- new net VoltSensor_2: J6.2, U2.14 (X1)
- new net VoltSensor_3: J6.3, U2.15 (X2)
- new net VoltSensor_4: J6.4, U2.12 (X3)
- new net VoltSensor_5: J6.5, U2.1 (X4)
- new net VoltSensor_6: J6.6, U2.5 (X5)
- no-connect marks 31 -> 25
Other:
- moved on the sheet: J1, J2, J3, R2, R4, R5

Commit message: 10/18/2023
Parts:
- added U4: OPA277P, OPA277P:DIP794W45P254L959H508Q8, symbol OPA277P:OPA277P
Changed lines of the file:
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@@
+    )
+  )
+  (symbol (lib_id "OPA277P:OPA277P") (at 255.27 184.15 0) (unit 1)
+    (in_bom yes) (on_board yes) (dnp no) (fields_autoplaced)
+    (property "Reference" "U4" (at 246.38 163.83 0)
+      (effects (font (size 1.27 1.27)))
+    )
+    (property "Value" "OPA277P" (at 246.38 166.37 0)
+      (effects (font (size 1.27 1.27)))
+    )
+    (property "Footprint" "OPA277P:DIP794W45P254L959H508Q8" (at 255.27 184.15 0)
+      (effects (font (size 1.27 1.27)) (justify bottom) hide)
+    )
+    (property "Datasheet" "" (at 255.27 184.15 0)
+      (effects (font (size 1.27 1.27)) hide)
+    )
+    (property "MF" "Texas Instruments" (at 255.27 184.15 0)
+      (effects (font (size 1.27 1.27)) (justify bottom) hide)
+    )
+    (property "Description" "\nDual, 36-V, 10&micro;V offset, 0.1&micro;V/˚C drift, bipolar, operational amplifier\n" (at 255.27 184.15 0)
+      (effects (font (size 1.27 1.27)) (justify bottom) hide)
+    )
+    (property "Package" "PDIP-8 Texas" (at 255.27 184.15 0)
+      (effects (font (size 1.27 1.27)) (justify bottom) hide)
+    )
+    (property "Price" "None" (at 255.27 184.15 0)
+      (effects (font (size 1.27 1.27)) (justify bottom) hide)
+    )
+    (property "SnapEDA_Link" "https://www.snapeda.com/parts/OPA277P/Texas+Instruments/view-part/?ref=snap" (at 255.27 184.15 0)
+      (effects (font (size 1.27 1.27)) (justify bottom) hide)
+    )
+    (property "MP" "OPA277P" (at 255.27 184.15 0)
+      (effects (font (size 1.27 1.27)) (justify bottom) hide)
+    )
+    (property "Purchase-URL" "https://www.snapeda.com/api/url_track_click_mouser/?unipart_id=1237537&manufacturer=Texas Instruments&part_name=OPA277P&search_term=opa277" (at 255.27 184.15 0)
+      (effects (font (size 1.27 1.27)) (justify bottom) hide)
+    )
+    (property "Availability" "In Stock" (at 255.27 184.15 0)
+      (effects (font (size 1.27 1.27)) (justify bottom) hide)
+    )
+    (property "Check_prices" "https://www.snapeda.com/parts/OPA277P/Texas+Instruments/view-part/?ref=eda" (at 255.27 184.15 0)
+      (effects (font (size 1.27 1.27)) (justify bottom) hide)
+    )
+    (pin "1")
+    (pin "2")
+    (pin "3")
+    (pin "4")
+    (pin "6")
+    (pin "7")
+    (pin "8")
+    (instances
+      (project "SeniorDesign"
+        (path "/24e33b4c-59d4-4763-9563-27915517cfab"
+          (reference "U4") (unit 1)
+        )
+      )
     )
   )

Commit message: 10/18/2023
Parts:
- removed C12: C, symbol Device:C
- added R3: 100k, symbol Device:R
Connections:
- net GND: now also R3.2
- net at U4.2 (-IN): now also U4.6 (OUTPUT)
- net at U4.3 (+IN): now also U2.3 (X), R3.1
- no-connect marks 25 -> 27
Other:
- moved on the sheet: U4
Changed lines of the file:
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@@
   (junction (at 162.56 198.12) (diameter 0) (color 0 0 0 0)
+  )
+  (junction (at 200.66 176.53) (diameter 0) (color 0 0 0 0)
   )
   (junction (at 234.95 25.4) (diameter 0) (color 0 0 0 0)
@@
   (no_connect (at 187.96 72.39))
   (no_connect (at 187.96 102.87))
+  (no_connect (at 212.09 181.61))
+  (no_connect (at 212.09 184.15))
   (no_connect (at 187.96 77.47))
   (no_connect (at 187.96 69.85))
@@
     (stroke (width 0) (type default))
   )
+  (wire (pts (xy 200.66 176.53) (xy 212.09 176.53))
+    (stroke (width 0) (type default))
+  )
   (polyline (pts (xy 52.07 15.24) (xy 52.07 45.72))
     (stroke (width 0) (type default))
@@
     (stroke (width 0) (type default))
   )
+  (wire (pts (xy 245.11 179.07) (xy 240.03 179.07))
+    (stroke (width 0) (type default))
+  )
   (wire (pts (xy 208.28 33.02) (xy 205.74 33.02))
     (stroke (width 0) (type default))
@@
     (stroke (width 0) (type default))
   )
+  (wire (pts (xy 200.66 190.5) (xy 200.66 187.96))
+    (stroke (width 0) (type default))
+  )
   (wire (pts (xy 234.95 27.94) (xy 234.95 25.4))
     (stroke (width 0) (type default))
@@
     (stroke (width 0) (type default))
   )
+  (wire (pts (xy 190.5 176.53) (xy 200.66 176.53))
+    (stroke (width 0) (type default))
+  )
   (wire (pts (xy 137.16 25.4) (xy 148.59 25.4))
     (stroke (width 0) (type default))
@@
     (stroke (width 0) (type default))
   )
+  (wire (pts (xy 245.11 189.23) (xy 245.11 179.07))
+    (stroke (width 0) (type default))
+  )
   (wire (pts (xy 146.05 81.28) (xy 139.7 81.28))
     (stroke (width 0) (type default))
@@
     (stroke (width 0) (type default))
   )
+  (wire (pts (xy 200.66 180.34) (xy 200.66 176.53))
+    (stroke (width 0) (type default))
+  )
   (wire (pts (xy 161.29 38.1) (xy 148.59 38.1))
     (stroke (width 0) (type default))
@@
     (stroke (width 0) (type default))
   )
+  (wire (pts (xy 209.55 179.07) (xy 209.55 189.23))
+    (stroke (width 0) (type default))
+  )
   (wire (pts (xy 186.69 38.1) (xy 173.99 38.1))
     (stroke (width 0) (type default))
@@
     (stroke (width 0) (type default))
   )
+  (wire (pts (xy 209.55 189.23) (xy 245.11 189.23))
+    (stroke (width 0) (type default))
+  )
   (wire (pts (xy 54.61 59.69) (xy 54.61 71.12))
     (stroke (width 0) (type default))
@@
   )
   (wire (pts (xy 162.56 189.23) (xy 162.56 191.77))
+    (stroke (width 0) (type default))
+  )
+  (wire (pts (xy 212.09 179.07) (xy 209.55 179.07))
     (stroke (width 0) (type default))
   )
@@
     )
   )
-  (symbol (lib_id "OPA277P:OPA277P") (at 255.27 184.15 0) (unit 1)
-    (in_bom yes) (on_board yes) (dnp no) (fields_autoplaced)
-    (property "Reference" "U4" (at 246.38 163.83 0)
-      (effects (font (size 1.27 1.27)))
-    )
-    (property "Value" "OPA277P" (at 246.38 166.37 0)
-      (effects (font (size 1.27 1.27)))
-    )
-    (property "Footprint" "OPA277P:DIP794W45P254L959H508Q8" (at 255.27 184.15 0)
-      (effects (font (size 1.27 1.27)) (justify bottom) hide)
-    )
-    (property "Datasheet" "" (at 255.27 184.15 0)
-      (effects (font (size 1.27 1.27)) hide)
-    )
-    (property "MF" "Texas Instruments" (at 255.27 184.15 0)
-      (effects (font (size 1.27 1.27)) (justify bottom) hide)
-    )
-    (property "Description" "\nDual, 36-V, 10&micro;V offset, 0.1&micro;V/˚C drift, bipolar, operational amplifier\n" (at 255.27 184.15 0)
-      (effects (font (size 1.27 1.27)) (justify bottom) hide)
-    )
-    (property "Package" "PDIP-8 Texas" (at 255.27 184.15 0)
-      (effects (font (size 1.27 1.27)) (justify bottom) hide)
-    )
-    (property "Price" "None" (at 255.27 184.15 0)
-      (effects (font (size 1.27 1.27)) (justify bottom) hide)
-    )
-    (property "SnapEDA_Link" "https://www.snapeda.com/parts/OPA277P/Texas+Instruments/view-part/?ref=snap" (at 255.27 184.15 0)
-      (effects (font (size 1.27 1.27)) (justify bottom) hide)
-    )
-    (property "MP" "OPA277P" (at 255.27 184.15 0)
-      (effects (font (size 1.27 1.27)) (justify bottom) hide)
-    )
-    (property "Purchase-URL" "https://www.snapeda.com/api/url_track_click_mouser/?unipart_id=1237537&manufacturer=Texas Instruments&part_name=OPA277P&search_term=opa277" (at 255.27 184.15 0)
-      (effects (font (size 1.27 1.27)) (justify bottom) hide)
-    )
-    (property "Availability" "In Stock" (at 255.27 184.15 0)
-      (effects (font (size 1.27 1.27)) (justify bottom) hide)
-    )
-    (property "Check_prices" "https://www.snapeda.com/parts/OPA277P/Texas+Instruments/view-part/?ref=eda" (at 255.27 184.15 0)
+  (symbol (lib_id "OPA277P:OPA277P") (at 234.95 189.23 0) (unit 1)
+    (in_bom yes) (on_board yes) (dnp no) (fields_autoplaced)
+    (property "Reference" "U4" (at 226.06 168.91 0)
+      (effects (font (size 1.27 1.27)))
+    )
+    (property "Value" "OPA277P" (at 226.06 171.45 0)
+      (effects (font (size 1.27 1.27)))
+    )
+    (property "Footprint" "OPA277P:DIP794W45P254L959H508Q8" (at 234.95 189.23 0)
+      (effects (font (size 1.27 1.27)) (justify bottom) hide)
+    )
+    (property "Datasheet" "" (at 234.95 189.23 0)
+      (effects (font (size 1.27 1.27)) hide)
+    )
+    (property "MF" "Texas Instruments" (at 234.95 189.23 0)
+      (effects (font (size 1.27 1.27)) (justify bottom) hide)
+    )
+    (property "Description" "\nDual, 36-V, 10&micro;V offset, 0.1&micro;V/˚C drift, bipolar, operational amplifier\n" (at 234.95 189.23 0)
+      (effects (font (size 1.27 1.27)) (justify bottom) hide)
+    )
+    (property "Package" "PDIP-8 Texas" (at 234.95 189.23 0)
+      (effects (font (size 1.27 1.27)) (justify bottom) hide)
+    )
+    (property "Price" "None" (at 234.95 189.23 0)
+      (effects (font (size 1.27 1.27)) (justify bottom) hide)
+    )
+    (property "SnapEDA_Link" "https://www.snapeda.com/parts/OPA277P/Texas+Instruments/view-part/?ref=snap" (at 234.95 189.23 0)
+      (effects (font (size 1.27 1.27)) (justify bottom) hide)
+    )
+    (property "MP" "OPA277P" (at 234.95 189.23 0)
+      (effects (font (size 1.27 1.27)) (justify bottom) hide)
+    )
+    (property "Purchase-URL" "https://www.snapeda.com/api/url_track_click_mouser/?unipart_id=1237537&manufacturer=Texas Instruments&part_name=OPA277P&search_term=opa277" (at 234.95 189.23 0)
+      (effects (font (size 1.27 1.27)) (justify bottom) hide)
+    )
+    (property "Availability" "In Stock" (at 234.95 189.23 0)
+      (effects (font (size 1.27 1.27)) (justify bottom) hide)
+    )
+    (property "Check_prices" "https://www.snapeda.com/parts/OPA277P/Texas+Instruments/view-part/?ref=eda" (at 234.95 189.23 0)
       (effects (font (size 1.27 1.27)) (justify bottom) hide)
     )
@@
         (path "/24e33b4c-59d4-4763-9563-27915517cfab"
           (reference "C15") (unit 1)
+        )
+      )
+    )
+  )
+  (symbol (lib_id "power:GND") (at 200.66 190.5 0) (unit 1)
+    (in_bom yes) (on_board yes) (dnp no)
+    (property "Reference" "#PWR028" (at 200.66 196.85 0)
+      (effects (font (size 1.27 1.27)) hide)
+    )
+    (property "Value" "GND" (at 200.66 195.58 0)
+      (effects (font (size 1.27 1.27)))
+    )
+    (property "Footprint" "" (at 200.66 190.5 0)
+      (effects (font (size 1.27 1.27)) hide)
+    )
+    (property "Datasheet" "" (at 200.66 190.5 0)
+      (effects (font (size 1.27 1.27)) hide)
+    )
+    (pin "1")
+    (instances
+      (project "SeniorDesign"
+        (path "/24e33b4c-59d4-4763-9563-27915517cfab"
+          (reference "#PWR028") (unit 1)
         )
       )
@@
     )
   )
-  (symbol (lib_id "Device:C") (at 88.9 167.64 0) (unit 1)
-    (in_bom yes) (on_board yes) (dnp no) (fields_autoplaced)
-    (property "Reference" "C12" (at 92.71 166.37 0)
-      (effects (font (size 1.27 1.27)) (justify left))
-    )
-    (property "Value" "C" (at 92.71 168.91 0)
-      (effects (font (size 1.27 1.27)) (justify left))
-    )
-    (property "Footprint" "" (at 89.8652 171.45 0)
-      (effects (font (size 1.27 1.27)) hide)
-    )
-    (property "Datasheet" "~" (at 88.9 167.64 0)
-      (effects (font (size 1.27 1.27)) hide)
-    )
-    (pin "1")
-    (pin "2")
-    (instances
-      (project "SeniorDesign"
-        (path "/24e33b4c-59d4-4763-9563-27915517cfab"
-          (reference "C12") (unit 1)
-        )
-      )
-    )
-  )
   (symbol (lib_id "Device:C") (at 222.25 31.75 0) (unit 1)
     (in_bom yes) (on_board yes) (dnp no) (fields_autoplaced)
@@
         )
       )
+    )
+  )
+  (symbol (lib_id "Device:R") (at 200.66 184.15 0) (unit 1)
+    (in_bom yes) (on_board yes) (dnp no) (fields_autoplaced)
+    (property "Reference" "R3" (at 203.2 182.88 0)
+      (effects (font (size 1.27 1.27)) (justify left))
+    )
+    (property "Value" "100k" (at 203.2 185.42 0)
+      (effects (font (size 1.27 1.27)) (justify left))
+    )
+    (property "Footprint" "" (at 198.882 184.15 90)
+      (effects (font (size 1.27 1.27)) hide)
+    )
+    (property "Datasheet" "~" (at 200.66 184.15 0)
+      (effects (font (size 1.27 1.27)) hide)
+    )
+    (pin "1")
+    (pin "2")
+    (instances
+      (project "SeniorDesign"
+        (path "/24e33b4c-59d4-4763-9563-27915517cfab"
+          (reference "R3") (unit 1)
+        )
+      )

Commit message: 10/18/2023 7:16PM
Parts:
- added C12, C18: 100n, symbol Device:C
- D2: value 1N47xxA -> 1N4728A
Connections:
- net +12V: now also U4.7 (V+), C18.1
- net -12V: now also U4.4 (V-), C12.2
- net GND: now also C12.1, C18.2
- net UART_RX: now also J3.3 (Pin_3); no longer J3.2 (Pin_2)
- net UART_TX: now also J3.2 (Pin_2); no longer J3.3 (Pin_3)
Other:
- moved on the sheet: J3

Commit message: 10/18/2023 7:22PM
Parts:
- added C13, C19: C, symbol Device:C
- added J7: 691243300007, 691243300007:691243300007, symbol 691243300007:691243300007
- added U7: OPA277P, OPA277P:DIP794W45P254L959H508Q8, symbol OPA277P:OPA277P
- added U8: CD4051B, symbol Analog_Switch:CD4051B
Connections:
- net +12V: now also C13.2, U7.7 (V+), U8.16 (VDD)
- net -12V: now also C19.1, U8.7 (VEE)
- net CurrSensor_1: now also J7.1, U7.3 (+IN)
- net CurrSensor_2: now also J7.2
- net CurrSensor_3: now also J7.3
- net CurrSensor_4: now also J7.4
- net CurrSensor_5: now also J7.5
- net CurrSensor_6: now also J7.6
- net GND: now also C13.1, C19.2, J7.7, U8.4 (X7), U8.6 (INH), U8.8 (VSS)
- new net: U7.2 (-IN), U7.6 (OUTPUT)
- new net CurrMux_0: U8.13 (X0)
- no-connect marks 27 -> 29
Other:
- moved on the sheet: C12, C18, J6, R3, U2, U4

Commit message: 10/24/2023 2:41PM
Parts:
- removed J4: 691243300007, 691243300007:691243300007, symbol 691243300007:691243300007
- removed U6, U8: CD4051B, symbol Analog_Switch:CD4051B
- added Amplifier1, U10, U11, U12, U14, U15, U8, U9: OPA277P, OPA277P:DIP794W45P254L959H508Q8, symbol OPA277P:OPA277P
- added C20, C21, C22, C25, C26, C27, C28, C29, C30, C31, C32, C33, C34, C35, C36, C37: 100n, symbol Device:C
- added D4, D5: 1N4007, Diode_THT:D_DO-41_SOD81_P10.16mm_Horizontal, symbol Diode:1N4007
- added R10: 157k, symbol Device:R
- added R11, R12, R14, R9: 1k, symbol Device:R
- added R13: 2k, symbol Device:R
- added R8: 100k, symbol Device:R
- added U13: CD4051B, symbol Analog_Switch:CD4051B
- C13, C19: value C -> 100n
Connections:
- net CurrSensor_6 is gone; now on net CurrSensor_5: J7.6
- net +12V: now also C13.1, Amplifier1.7 (V+), C20.1, C22.1, C26.1, C28.1, C30.1, C32.1, C34.1, C36.1, U10.7 (V+), U11.7 (V+), U12.7 (V+), U13.16 (VDD), U14.7 (V+), U15.7 (V+), U8.7 (V+), U9.7 (V+); no longer C13.2
- net -12V: now also C19.2, U7.4 (V-), Amplifier1.4 (V-), C21.2, C25.2, C27.2, C29.2, C31.2, C33.2, C35.2, C37.2, U10.4 (V-), U11.4 (V-), U12.4 (V-), U13.7 (VEE), U14.4 (V-), U15.4 (V-), U8.4 (V-), U9.4 (V-); no longer C19.1
- net CurrMux_0: now also U7.2 (-IN), U7.6 (OUTPUT), U13.13 (X0)
- net CurrSensor_1: now also J7.2, U8.3 (+IN); no longer J7.1, U7.3 (+IN)
- net CurrSensor_2: now also J7.3, U9.3 (+IN); no longer J7.2
- net CurrSensor_3: now also J7.4, U10.3 (+IN); no longer J7.3
- net CurrSensor_4: now also J7.5, U11.3 (+IN); no longer J7.4
- net CurrSensor_5: now also U12.3 (+IN); no longer J7.5
- net GND: now also C13.2, C19.1, Amplifier1.3 (+IN), C20.2, C21.1, C22.2, C25.1, C26.2, C27.1, C28.2, C29.1, C30.2, C31.1, C32.2, C33.1, C34.2, C35.1, C36.2, C37.1, R14.1, R8.2, U13.2 (X6), U13.4 (X7), U13.6 (INH), U13.8 (VSS), U15.3 (+IN); no longer C13.1, C19.2
- net GPIO_A: now also U13.11 (A)
- net GPIO_B: now also U13.10 (B)
- net GPIO_C: now also U13.9 (C)
- new net: D4.2 (A), R11.2, R12.1, U15.2 (-IN)
- new net: Amplifier1.2 (-IN), R10.1, R9.2
- new net: D4.1 (K), D5.2 (A), U15.6 (OUTPUT)
- new net CurrADC: R13.1, R14.2
- new net CurrAmp: Amplifier1.6 (OUTPUT), R10.2, R11.1
- new net CurrMuxOp: R8.1, U13.3 (X), U14.3 (+IN)
- new net CurrMux_1: U13.14 (X1), U8.2 (-IN), U8.6 (OUTPUT)
- new net CurrMux_2: U13.15 (X2), U9.2 (-IN), U9.6 (OUTPUT)
- new net CurrMux_3: U10.2 (-IN), U10.6 (OUTPUT), U13.12 (X3)
- new net CurrMux_4: U11.2 (-IN), U11.6 (OUTPUT), U13.1 (X4)
- new net CurrMux_5: U12.2 (-IN), U12.6 (OUTPUT), U13.5 (X5)
- new net CurrPreAmp: R9.1, U14.2 (-IN), U14.6 (OUTPUT)
- new net CurrRect: D5.1 (K), R12.2, R13.2
- new net CurrSensor_0: J7.1, U7.3 (+IN)
- no-connect marks 29 -> 45
Other:
- note added: "Current Sensor"
- moved on the sheet: C12, C18, J6, R3, U2, U4

Commit message: 10/26/2023
Parts:
- removed J2, J3: Conn_01x04_Pin, symbol Connector:Conn_01x04_Pin
- removed J5: XLR6, symbol Connector_Audio:XLR6
- removed J6, J7: 691243300007, 691243300007:691243300007, symbol 691243300007:691243300007
- added C38, C39: 100n, Capacitor_SMD:C_0603_1608Metric, symbol Device:C
- added D6, D7: 1N4007, Diode_THT:D_DO-41_SOD81_P10.16mm_Horizontal, symbol Diode:1N4007
- added H2: MountingHole_Pad, MountingHole:MountingHole_2.2mm_M2, symbol Mechanical:MountingHole_Pad
- added Q1, Q2, Q3: 2N2222, 2N2222:TO127P584H533-3, symbol 2N2222:2N2222
- added R15, R16, R19, R20, R21: 1k, Resistor_SMD:R_0603_1608Metric, symbol Device:R
- added R17: 270k, Resistor_SMD:R_0603_1608Metric, symbol Device:R
- added R18: 100k, Resistor_SMD:R_0603_1608Metric, symbol Device:R
- added R22, R23, R24: 2k, Resistor_SMD:R_0603_1608Metric, symbol Device:R
- added U17, U18, U19, U20: 282836-7, 282836-7_TYC, symbol 282836_7:282836-7
- added U6: OPA277P, OPA277P:DIP794W45P254L959H508Q8, symbol OPA277P:OPA277P
- C1, C10, C11, C12, C13, C14, C15, C16, C17, C18, C19, C2, C20, C21, C22, C25, C26, C27, C28, C29, C3, C30, C31, C32, C33, C34, C35, C36, C37, C4, C5, C6, C7, C8, C9: footprint (none) -> Capacitor_SMD:C_0603_1608Metric
- C23, C24: footprint (none) -> Capacitor_SMD:CP_Elec_4x5.4
- FB1: footprint (none) -> Inductor_SMD:L_0603_1608Metric
- J1: footprint (none) -> Connector_USB:USB_Micro-B_Wuerth_629105150521
- R1, R10, R11, R12, R13, R14, R2, R3, R4, R5, R6, R7, R8, R9: footprint (none) -> Resistor_SMD:R_0603_1608Metric
- SW1: footprint (none) -> Button_Switch_SMD:SW_SPDT_PCM12
- U13, U2: footprint (none) -> CD4051BM96:D16
- U5: footprint (none) -> Package_TO_SOT_THT:TO-220-3_Vertical
- Y1: footprint (none) -> Crystal:Crystal_SMD_3225-4Pin_3.2x2.5mm
- renumbered Amplifier1 to U16
Connections:
- net CurrADC is gone; now on net ADC1_IN6: R13.1, R14.2
- net +12V: now also C38.1, R22.2, R23.2, R24.2, U6.7 (V+)
- net +15V: now also U17.1
- net +3V3: now also U18.1; no longer C6.1, C7.1, FB1.1, U1.9 (VDDA)
- net -12V: now also C39.2, U6.4 (V-)
- net -15V: now also U17.2
- net ADC2_IN9: now also R17.2, R18.1
- net CurrSensor_0: now also U19.1
- net CurrSensor_1: now also U19.2
- net CurrSensor_2: now also U19.3
- net CurrSensor_3: now also U19.4
- net CurrSensor_4: now also U19.5
- net CurrSensor_5: now also U19.6
- net GND: now also C38.2, C39.1, Q1.1, Q2.1, Q3.1, R18.2, U17.7, U18.7, U19.7, U20.7, U6.3 (+IN)
- net GPIO_A: now also R19.1; no longer U13.11 (A), U2.11 (A)
- net GPIO_B: now also R20.1; no longer U13.10 (B), U2.10 (B)
- net GPIO_C: now also R21.1; no longer U13.9 (C), U2.9 (C)
- net SWCLK: now also U18.4
- net SWDIO: now also U18.5
- net UART_RX: now also U1.43 (PB7), U18.3; no longer U1.13 (PA3)
- net UART_TX: now also U1.42 (PB6), U18.2; no longer U1.12 (PA2)
- net USB_D+: now also R2.2
- net USB_D-: no longer R2.2
- net VoltSensor_1: now also U20.1
- net VoltSensor_2: now also U20.2
- net VoltSensor_3: now also U20.3
- net VoltSensor_4: now also U20.4
- net VoltSensor_5: now also U20.5
- net VoltSensor_6: now also U20.6
- net Volt_Amp: now reaches U4.2 (-IN), U4.6 (OUTPUT)
- net Volt_Amp: now also R15.1
- net TIM2_CH1: no longer names the net of U1.10 (PA0)
- new net: Q1.2, R19.2
- new net: D7.1 (K), R16.2, R17.1
- new net: D6.1 (K), D7.2 (A), U6.6 (OUTPUT)
- new net: Q3.2, R21.2
- new net: D6.2 (A), R15.2, R16.1, U6.2 (-IN)
- new net: Q2.2, R20.2
- new net +3.3VA: C6.1, C7.1, FB1.1, U1.9 (VDDA)
- new net MUX_A: Q1.3, R22.1, U13.11 (A), U2.11 (A)
- new net MUX_B: Q2.3, R23.1, U13.10 (B), U2.10 (B)
- new net MUX_C: Q3.3, R24.1, U13.9 (C), U2.9 (C)
- no-connect marks 45 -> 52
Other:
- note added: "Communication"
- note added: "Mux Selectors"
- note added: "Voltage Sensor"
- moved on the sheet: C1, C10, C11, C12, C13, C14, C15, C16, C17, C18, C19, C2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
