File: SeniorDesign.kicad_pcb (KiCad board)
At the start: 4 copper layers, 101 parts, among them J1 USB_B_Micro, Q1 2N2222, Q2 2N2222, Q3 2N2222, SW1 SW_SPDT, U1 STM32F103C8Tx, U10 OPA277P, U11 OPA277P, U12 OPA277P, U13 CD4051B, U14 OPA277P, U15 OPA277P, U16 OPA277P, U17 282836-7, U18 282836-7, U19 282836-7, U2 CD4051B, U20 282836-7, U3 LM7812_TO220, U4 OPA277P, U5 L7912, U6 OPA277P, U7 OPA277P, U8 OPA277P, U9 OPA277P, Y1 16MHz

Commit message: 10/26/2023
Parts:
- moved Q3 117.1 mm to (76.8, 40.2), turned to 90 degrees
- moved R24 114.6 mm to (71.2, 39.0), turned to 180 degrees
- moved R23 103.9 mm to (71.2, 48.0), turned to 180 degrees
- moved Q2 101.9 mm to (76.8, 49.2), turned to 90 degrees
- moved R22 93.6 mm to (71.2, 56.8), turned to 180 degrees
- moved Q1 87.5 mm to (76.8, 58.0), turned to 90 degrees
- moved R21 80.4 mm to (72.5, 68.5), turned to 90 degrees
- moved R20 77.2 mm to (74.5, 68.5), turned to 90 degrees
- moved R19 74.0 mm to (76.5, 68.5), turned to 90 degrees
- moved SW1 53.2 mm to (34.8, 21.5), turned to 180 degrees
- moved R6 24.1 mm to (55.2, 54.5), turned to 90 degrees
- moved R7 21.5 mm to (56.0, 49.2), turned to 0 degrees
- moved D2 18.0 mm to (55.2, 59.2), turned to -90 degrees
- moved J1 3.47 mm to (89.7, 77.8)
- moved H2 3.16 mm to (89.0, 24.0)
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Other:
- board outline added: 74.2 x 148.8 mm

Commit message: 10/26/2023
Parts:
- moved R7 5.53 mm to (57.8, 54.5), turned to 90 degrees
- moved C10 3.27 mm to (58.5, 82.8), turned to 180 degrees
- moved C11 3.27 mm to (58.5, 76.2), turned to 0 degrees
- moved R2 2.77 mm to (83.2, 76.5)
- moved C9 2.04 mm to (65.8, 89.0), turned to 180 degrees
- moved C4 1.67 mm to (78.8, 75.0)
- moved C6 1.08 mm to (64.2, 80.8)
- moved C23 0.58 mm to (53.5, 42.2)
- moved R5 0.50 mm to (80.8, 79.8)
- moved R13 0.25 mm to (72.8, 88.5)
- turned R6 to -90 degrees
Routing:
- net /SW_BOOT0: track 0.00 -> 74.8 mm, vias 0 -> 2
- net GND: track 0.00 -> 57.5 mm, vias 0 -> 29
- net +15V: track 0.00 -> 39.0 mm
- net +3V3: track 0.00 -> 20.3 mm
- net -15V: track 0.00 -> 14.7 mm
- net /NRST: track 0.00 -> 13.8 mm, vias 0 -> 1
- net /HSE_IN: track 0.00 -> 12.8 mm
- net /USB_D+: track 0.00 -> 12.6 mm
- net /USB_D-: track 0.00 -> 12.2 mm
- net /HSE_OUT: track 0.00 -> 10.9 mm
- net /BOOT0: track 0.00 -> 8.91 mm
- net +3.3VA: track 0.00 -> 8.26 mm
- net /VBUS_SENSE: track 0.00 -> 8.01 mm
- net Net-(D1-A): track 0.00 -> 7.23 mm
- net /GPIO_A: track 0.00 -> 6.85 mm
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- added copper zone on F.Cu, net +12V
- added copper zone on In2.Cu, net +12V
- added copper zone on F.Cu, net +3V3
- added copper zone on F.Cu, net GND
- added copper zone on In1.Cu, net GND

Commit message: 10/27/2023
Parts:
- moved Q1 19.3 mm to (77.5, 38.8)
- moved R22 19.3 mm to (72.0, 37.5)
- moved Q3 18.5 mm to (77.5, 58.8)
- moved R24 18.5 mm to (72.0, 57.5)
- moved R18 3.93 mm to (60.0, 90.8), turned to 90 degrees
- moved R16 2.00 mm to (50.5, 94.2)
- moved D6 1.76 mm to (49.8, 107.1)
- moved C25 1.27 mm to (61.8, 133.5), turned to 0 degrees
- moved C19 1.13 mm to (34.0, 123.5), turned to 0 degrees
- moved C27 1.13 mm to (34.0, 138.5), turned to 0 degrees
- moved C29 1.13 mm to (48.0, 143.5), turned to 0 degrees
- moved C31 1.13 mm to (62.0, 148.5), turned to 0 degrees
- moved C21 1.08 mm to (47.8, 128.5), turned to 0 degrees
- moved Q2 0.90 mm to (77.5, 48.8)
- moved R23 0.90 mm to (72.0, 47.5)
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Routing:
- net -12V: track 6.11 -> 243.1 mm, vias 0 -> 13
- net +3V3: track 20.3 -> 121.6 mm, vias 0 -> 5
- net GND: track 57.5 -> 119.5 mm, vias 29 -> 54
- net /MUX_A: track 0.00 -> 54.5 mm, vias 0 -> 2
- net /MUX_B: track 0.00 -> 43.7 mm, vias 0 -> 2
- net /SWDIO: track 0.00 -> 41.4 mm, vias 0 -> 2
- net /CurrSensor_2: track 0.00 -> 38.8 mm, vias 0 -> 1
- net /CurrSensor_5: track 0.00 -> 37.8 mm
- net /MUX_C: track 0.00 -> 34.2 mm, vias 0 -> 2
- net +12V: track 3.27 -> 36.8 mm, vias 10 -> 19
- net Net-(Q1-Pad2): track 0.00 -> 33.4 mm
- net /SWCLK: track 0.00 -> 30.0 mm
- net /UART_RX: track 0.00 -> 29.8 mm, vias 0 -> 2
- net /VoltSensor_6: track 0.00 -> 27.0 mm, vias 0 -> 1
- net Net-(Q2-Pad2): track 0.00 -> 24.4 mm
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- added copper zone on F.Cu, net -12V

Commit message: 10/30/2023 12:00AM
Parts:
- Current Sensors: renamed from U19
- Voltage Sensors: renamed from U20
- moved R11 1.22 mm to (75.0, 101.2)
- moved R13 0.88 mm to (73.5, 89.0)
- moved C33 0.50 mm to (71.8, 107.8)
- moved C34 0.25 mm to (71.8, 97.0)
- moved C32 0.25 mm to (59.3, 114.2)
- moved C36 0.25 mm to (88.3, 101.5)
- moved C37 0.25 mm to (75.8, 106.5)
- renumbered U18 to Communication, U17 to Power
Routing:
- net /CurrMux_0: track 8.99 -> 122.0 mm, vias 0 -> 4
- net /CurrMux_1: track 8.99 -> 104.0 mm, vias 0 -> 2
- net /CurrMux_3: track 8.99 -> 101.9 mm, vias 0 -> 2
- net /MUX_A: track 54.5 -> 142.1 mm, vias 2 -> 4
- net /MUX_B: track 43.7 -> 126.8 mm, vias 2 -> 4
- net -12V: track 243.1 -> 326.3 mm, vias 13 -> 15
- net /MUX_C: track 34.2 -> 109.9 mm, vias 2 -> 4
- net +3V3: track 121.6 -> 180.8 mm, vias 5 -> 7
- net /CurrMux_4: track 8.99 -> 51.2 mm, vias 0 -> 4
- net /CurrMux_5: track 8.99 -> 44.0 mm, vias 0 -> 2
- net /CurrMux_2: track 8.99 -> 43.9 mm, vias 0 -> 2
- net GND: track 119.5 -> 142.2 mm, vias 54 -> 63
- net Net-(D4-A): track 0.00 -> 18.3 mm
- net Net-(D4-K): track 0.00 -> 17.9 mm
- net Net-(U16--IN): track 0.00 -> 17.2 mm
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
Commit message: 11/3/2023 12:42AM
Parts:
- removed the C19 at (34.0, 123.5)
- removed the C20 at (61.0, 122.8)
- removed the C21 at (47.8, 128.5)
- removed the C22 at (75.0, 127.8)
- removed the C37 at (75.8, 106.5)
- removed the D2 at (55.2, 59.2)
- removed the H2 at (89.0, 162.8)
- removed the H2 at (24.8, 162.8)
- removed the H2 at (24.8, 24.0)
- removed the R6 at (55.2, 54.5)
- removed the R7 at (57.8, 54.5)
- added C10: 22uf, Capacitor_SMD:C_0603_1608Metric, F.Cu at (62.8, 58.3)
- added C14: 100n, Capacitor_SMD:C_0603_1608Metric, F.Cu at (39.2, 92.2)
- added C15: 10uf, Capacitor_SMD:C_0603_1608Metric, F.Cu at (47.0, 92.2)
- added C16: 10uf, Capacitor_SMD:C_0603_1608Metric, F.Cu at (39.2, 76.2)
- added C17: 10uf, Capacitor_SMD:C_0603_1608Metric, F.Cu at (44.0, 106.0)
- added C18: 10uf, Capacitor_SMD:C_0603_1608Metric, F.Cu at (39.2, 90.5)
- added C3: 100u, Capacitor_SMD:C_0603_1608Metric, F.Cu at (52.5, 33.0)
- added C4: 100u, Capacitor_SMD:C_0603_1608Metric, F.Cu at (46.2, 34.2)
- added C40: 10uf, Capacitor_SMD:C_0603_1608Metric, F.Cu at (63.0, 122.8)
- added C41: 10uf, Capacitor_SMD:C_0603_1608Metric, F.Cu at (47.8, 130.0)
- added C42: 10uf, Capacitor_SMD:C_0603_1608Metric, F.Cu at (77.0, 127.8)
- added C43: 10uf, Capacitor_SMD:C_0603_1608Metric, F.Cu at (61.8, 135.0)
- added C44: 10uf, Capacitor_SMD:C_0603_1608Metric, F.Cu at (48.8, 133.2)
- added C45: 10uf, Capacitor_SMD:C_0603_1608Metric, F.Cu at (34.0, 140.2)
- added C46: 10uf, Capacitor_SMD:C_0603_1608Metric, F.Cu at (62.8, 137.8)
- added C47: 10uf, Capacitor_SMD:C_0603_1608Metric, F.Cu at (48.0, 141.8)
- added C48: 10uf, Capacitor_SMD:C_0603_1608Metric, F.Cu at (77.0, 142.8)
- added C49: 10uf, Capacitor_SMD:C_0603_1608Metric, F.Cu at (62.0, 146.8)
- added C54: 100n, Capacitor_SMD:C_0603_1608Metric, F.Cu at (59.2, 114.2)
- added C55: 100n, Capacitor_SMD:C_0603_1608Metric, F.Cu at (71.8, 107.8)
- added C56: 100n, Capacitor_SMD:C_0603_1608Metric, F.Cu at (71.8, 97.0)
- added C57: 100n, Capacitor_SMD:C_0603_1608Metric, F.Cu at (59.5, 102.0)
- added C58: 100n, Capacitor_SMD:C_0603_1608Metric, F.Cu at (88.0, 101.5)
- added C59: 100n, Capacitor_SMD:C_0603_1608Metric, F.Cu at (76.0, 106.5)
- added C60: 10uf, Capacitor_SMD:C_0603_1608Metric, F.Cu at (57.2, 114.2)
- added C61: 10uf, Capacitor_SMD:C_0603_1608Metric, F.Cu at (73.5, 109.2)
- added C62: 10uf, Capacitor_SMD:C_0603_1608Metric, F.Cu at (73.8, 97.0)
- added C63: 10uf, Capacitor_SMD:C_0603_1608Metric, F.Cu at (57.5, 102.0)
- added C64: 10uf, Capacitor_SMD:C_0603_1608Metric, F.Cu at (90.0, 101.5)
- added C65: 10uf, Capacitor_SMD:C_0603_1608Metric, F.Cu at (74.2, 106.0)
- added C66: 100u, Capacitor_SMD:C_0603_1608Metric, F.Cu at (58.0, 32.4)
- added C9: 10uf, Capacitor_SMD:C_0603_1608Metric, F.Cu at (62.0, 54.5)
- added Css1: 1nf, Capacitor_SMD:C_0603_1608Metric, F.Cu at (57.8, 54.8)
- added D10: SMAJ12CA, Diode_SMD:D_SMA, B.Cu at (24.2, 80.0)
- added D11: SMAJ12CA, Diode_SMD:D_SMA, B.Cu at (24.2, 85.0)
- added D12: SMAJ12CA, Diode_SMD:D_SMA, B.Cu at (24.2, 90.0)
- added D7: SMAJ12CA, Diode_SMD:D_SMA, B.Cu at (24.2, 75.2)
- added D8: SMAJ12CA, Diode_SMD:D_SMA, B.Cu at (24.2, 70.0)
- added D9: SMAJ12CA, Diode_SMD:D_SMA, B.Cu at (24.2, 65.2)
- added H2: MountingHole_Pad, MountingHole:MountingHole_2.2mm_M2, F.Cu at (24.5, 24.0)
- added H3: MountingHole_Pad, MountingHole:MountingHole_2.2mm_M2, F.Cu at (24.5, 162.8)
- added H4: MountingHole_Pad, MountingHole:MountingHole_2.2mm_M2, F.Cu at (89.0, 162.8)
- added R25: 0, Resistor_SMD:R_0603_1608Metric, F.Cu at (49.8, 57.2)
- added R26: 0, Resistor_SMD:R_0603_1608Metric, F.Cu at (56.2, 51.0)
- added R27: 0, Resistor_SMD:R_0603_1608Metric, F.Cu at (62.5, 61.5)
- added R4: 249k, Resistor_SMD:R_0603_1608Metric, F.Cu at (58.8, 60.0)
- added R5: 100k, Resistor_SMD:R_0603_1608Metric, F.Cu at (55.5, 59.2)
- added Rmode1: 40.2k, Resistor_SMD:R_0603_1608Metric, F.Cu at (58.8, 53.0)
- added U5: TPSM82902SISR, footprints:uSIP11_SIS_TEX, F.Cu at (60.0, 57.2)
- C38, C39: value 100n -> 10uf
- U1: renamed from Power; footprint footprints:282836-7_TYC -> 282836_7:282836-7_TYC
- U21: renamed from Communication; footprint footprints:282836-7_TYC -> 282836_7:282836-7_TYC
- U4: renamed from Voltage Sensors; footprint footprints:282836-7_TYC -> 282836_7:282836-7_TYC
- U9: renamed from Current Sensors; footprint footprints:282836-7_TYC -> 282836_7:282836-7_TYC
- moved C36 53.8 mm to (62.0, 148.5), turned to 0 degrees
- moved C34 52.2 mm to (48.0, 143.5), turned to 0 degrees
- moved C35 43.7 mm to (75.0, 142.8), turned to 90 degrees
- moved C32 35.0 mm to (34.0, 138.5), turned to 0 degrees
- moved C39 33.4 mm to (34.0, 125.0), turned to 0 degrees
- moved C33 31.9 mm to (61.0, 137.8), turned to 90 degrees
- moved C27 31.3 mm to (61.0, 122.8), turned to 90 degrees
- moved C29 31.3 mm to (75.0, 127.8), turned to 90 degrees
- moved C25 21.6 mm to (47.0, 117.8), turned to 90 degrees
- moved C31 21.4 mm to (47.0, 133.3), turned to 90 degrees
- moved C30 16.2 mm to (61.8, 133.5), turned to 0 degrees
- moved C28 16.2 mm to (47.8, 128.5), turned to 0 degrees
- moved C26 16.0 mm to (34.0, 123.5), turned to 0 degrees
- moved C38 14.2 mm to (49.0, 117.8), turned to 90 degrees
- moved C13 13.8 mm to (44.0, 104.2), turned to 0 degrees
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- renumbered C23 to C1, C18 to C11, C5 to C19, C14 to C2, C9 to C20, C11 to C21, C4 to C22, C10 to C23, C3 to C24, C2 to C37, C15 to C5, C1 to C50, C6 to C51, C7 to C52, C8 to C53, C16 to C6, C24 to C7, C17 to C8, D3 to D2, D6 to D3, D7 to D4, D4 to D5, D5 to D6, H2 to H1, R15 to R1, R21 to R10, R22 to R11, R23 to R12, R24 to R13, R1 to R14, R8 to R15, R9 to R16, R11 to R17, R2 to R18, R4 to R19, R3 to R2, R5 to R20, R10 to R21, R12 to R22, R13 to R23, R14 to R24, R16 to R3, R17 to R6, R18 to R7, R19 to R8, R20 to R9, U7 to U10, U8 to U11, U9 to U12, U10 to U13, U11 to U14, U12 to U15, U1 to U16, U13 to U17, U14 to U18, U16 to U19, U5 to U2, U15 to U20, U2 to U6, U4 to U7, U6 to U8
Connections:
- C25 pad 1: GND -> +12V
- C25 pad 2: -12V -> GND
- C26 pad 1: +12V -> GND
- C26 pad 2: GND -> -12V
- C27 pad 1: GND -> +12V
- C27 pad 2: -12V -> GND
- C28 pad 1: +12V -> GND
- C28 pad 2: GND -> -12V
- C29 pad 1: GND -> +12V
- C29 pad 2: -12V -> GND
- C30 pad 1: +12V -> GND
- C30 pad 2: GND -> -12V
- C31 pad 1: GND -> +12V
- C31 pad 2: -12V -> GND
- C32 pad 1: +12V -> GND
- C32 pad 2: GND -> -12V
- C33 pad 1: GND -> +12V
- C33 pad 2: -12V -> GND
- C34 pad 1: +12V -> GND
- C34 pad 2: GND -> -12V
- C35 pad 1: GND -> +12V
- C35 pad 2: -12V -> GND
- C36 pad 1: +12V -> GND
- C36 pad 2: GND -> -12V
- U1 pad 3: unconnected-(U17-Pad3) -> +5V
Routing:
- net GND: track 142.2 -> 182.5 mm, vias 63 -> 90
- net +5V: track 0.00 -> 27.9 mm, vias 0 -> 2
- net +12V: track 50.8 -> 76.6 mm, vias 23 -> 21
- net -12V: track 326.3 -> 344.1 mm
- net +3V3: track 180.8 -> 171.8 mm
- net /SW_BOOT0: track 74.8 -> 68.2 mm
- net /CurrMux_1: track 104.0 -> 108.7 mm
- net Net-(U5-PG): track 0.00 -> 3.44 mm
- net /CurrMux_2: track 43.9 -> 47.2 mm
- net /CurrMux_0: track 122.0 -> 125.3 mm
- net Net-(U5-MODE/S-CONF): track 0.00 -> 3.17 mm
- net Net-(D3-K): track 18.3 -> 21.4 mm
- net /VoltSensor_2: track 21.0 -> 18.8 mm
- net /VoltSensor_4: track 24.1 -> 21.9 mm
- net /VoltSensor_3: track 18.9 -> 16.7 mm
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- added copper zone on F.Cu, net +5V
- added copper zone on B.Cu, net /VoltSensor_1
- added copper zone on B.Cu, net /VoltSensor_2
- added copper zone on B.Cu, net /VoltSensor_3
- added copper zone on B.Cu, net /VoltSensor_4
- added copper zone on B.Cu, net /VoltSensor_5
- added copper zone on B.Cu, net /VoltSensor_6
- added copper zone on B.Cu, net GND
Other:
- board text added: "+15V"
- board text added: "+5V"
- board text added: "- Designed By - Michael Mederos Julio Barreto Tannoux"
- board text added: "-15V"
- board text added: "1"
- board text added: "2"
- board text added: "3"
- board text added: "3.3V"
- board text added: "4"
- board text added: "5"
- board text added: "6"
- board text added: "GND"
- board text added: "RX"
- board text added: "SWCLK"
- board text added: "SWDIO"
- board text added: "Senior Design (V1.0) Machine Learning Applications in Power System Fault Location with ADMS and AMI"
- board text added: "TX"
